Commit message: commit to launch

File: description/robot_core.xacro (robot description, xacro)
@@ -1,4 +1,4 @@
 <?xml version="1.0"?>
-<robot xmlns:xacro="http://www.ros.org/wiki/xacro"   >
+<robot xmlns:xacro="http://www.ros.org/wiki/xacro" name="my_robot">
     <xacro:include filename="inertial_macro.xacro"/>
     <material name="white">
@@ -14,25 +14,22 @@
         <color rgba="0 0 0 1"/>
     </material>
-<!--base_link-->
-    <link name = "base_link">
-    </link>
-<!--chassis_link-->
-    <joint name = "chassis_joint" type = "fixed">
-        <parent link = "base_link"/>
-        <child link = "chassis_link"/>
-        <origin xyz = "-0.10 0 0"/>
+    <link name="base_link"></link>
+    <joint name="chassis_joint" type="fixed">
+        <parent link="base_link"/>
+        <child link="chassis_link"/>
+        <origin xyz="-0.10 0 0"/>
     </joint>
-    <link name = "chassis_link">
+    <link name="chassis_link">
         <visual>
-            <origin xyz = "0.15 0 0.075"/>
+            <origin xyz="0.15 0 0.075"/>
             <geometry>
-                <box size = "0.3 0.3 0.15"/>
+                <box size="0.3 0.3 0.15"/>
             </geometry>
             <material name="white"/>
         </visual>
         <collision>
-            <origin xyz = "0.15 0 0.075"/>
+            <origin xyz="0.15 0 0.075"/>
             <geometry>
-                <box size = "0.3 0.3 0.15"/>
+                <box size="0.3 0.3 0.15"/>
             </geometry>
         </collision>
@@ -41,23 +38,31 @@
         </xacro:inertial_box>
     </link>
-<!--left wheel link -->
-    <joint name = "left_wheel_joint" type = "continuous">
-        <parent link = "base_link"/>
-        <child link = "left_wheel_link"/>
-        <origin xyz = "0.0 0.175 0" rpy = "-${pi/2} 0 0" />
-        <axis xyz = "0 0 1"/>
+    <gazebo reference="chassis_link">
+        <visual>
+            <material>
+                <ambient>1.0 0.0 0.0 1.0</ambient>
+                <diffuse>1.0 0.0 0.0 1.0</diffuse>
+                <specular>0.5 0.5 0.5 1.0</specular>
+            </material>
+        </visual>
+    </gazebo>
+    <joint name="left_wheel_joint" type="continuous">
+        <parent link="base_link"/>
+        <child link="left_wheel_link"/>
+        <origin xyz="0.0 0.175 0" rpy="-${pi/2} 0 0" />
+        <axis xyz="0 0 1"/>
     </joint>
-    <link name = "left_wheel_link">
+    <link name="left_wheel_link">
         <visual>
-            <origin xyz = "0 0 0"/>
+            <origin xyz="0 0 0"/>
             <geometry>
-                <cylinder radius = "0.05" length = "0.04"/>
+                <cylinder radius="0.05" length="0.04"/>
             </geometry>
             <material name="blue"/>
         </visual>
         <collision>
-            <origin xyz = "0 0 0"/>
+            <origin xyz="0 0 0"/>
             <geometry>
-                <cylinder radius = "0.05" length = "0.04"/>
+                <cylinder radius="0.05" length="0.04"/>
             </geometry>
         </collision>
@@ -66,23 +71,31 @@
         </xacro:inertial_cylinder>
     </link>
-    <!--right wheel link -->
-    <joint name = "right_wheel_joint" type = "continuous">
-        <parent link = "base_link"/>
-        <child link = "right_wheel_link"/>
-        <origin xyz = "0.0 -0.175 0" rpy = "${pi/2} 0 0" />
-        <axis xyz = "0 0 -1"/>
+    <gazebo reference="left_wheel_link">
+        <visual>
+            <material>
+                <ambient>0.0 0.0 1.0 1.0</ambient>
+                <diffuse>0.0 0.0 1.0 1.0</diffuse>
+                <specular>0.5 0.5 0.5 1.0</specular>
+            </material>
+        </visual>
+    </gazebo>
+    <joint name="right_wheel_joint" type="continuous">
+        <parent link="base_link"/>
+        <child link="right_wheel_link"/>
+        <origin xyz="0.0 -0.175 0" rpy="${pi/2} 0 0" />
+        <axis xyz="0 0 -1"/>
     </joint>
-    <link name = "right_wheel_link">
+    <link name="right_wheel_link">
         <visual>
-            <origin xyz = "0 0 0"/>
+            <origin xyz="0 0 0"/>
             <geometry>
-                <cylinder radius = "0.05" length = "0.04"/>
+                <cylinder radius="0.05" length="0.04"/>
             </geometry>
             <material name="blue"/>
         </visual>
         <collision>
-            <origin xyz = "0 0 0"/>
+            <origin xyz="0 0 0"/>
             <geometry>
-                <cylinder radius = "0.05" length = "0.04"/>
+                <cylinder radius="0.05" length="0.04"/>
             </geometry>
         </collision>
@@ -91,22 +104,30 @@
         </xacro:inertial_cylinder>
     </link>
-    <!--caster wheel link -->
-    <joint name = "caster_wheel_joint" type = "fixed">
-        <parent link = "chassis_link"/>
-        <child link = "caster_wheel_link"/>
-        <origin xyz = "0.24 0 0" />
+    <gazebo reference="right_wheel_link">
+        <visual>
+            <material>
+                <ambient>0.0 0.0 1.0 1.0</ambient>
+                <diffuse>0.0 0.0 1.0 1.0</diffuse>
+                <specular>0.5 0.5 0.5 1.0</specular>
+            </material>
+        </visual>
+    </gazebo>
+    <joint name="caster_wheel_joint" type="fixed">
+        <parent link="chassis_link"/>
+        <child link="caster_wheel_link"/>
+        <origin xyz="0.24 0 0" />
     </joint>
-    <link name = "caster_wheel_link">
+    <link name="caster_wheel_link">
         <visual>
-            <origin xyz = "0 0 0"/>
+            <origin xyz="0 0 0"/>
             <geometry>
-                <sphere radius = "0.05"/>
+                <sphere radius="0.05"/>
             </geometry>
             <material name="black"/>
         </visual>
          <collision>
-            <origin xyz = "0 0 0"/>
+            <origin xyz="0 0 0"/>
             <geometry>
-                <sphere radius = "0.05"/>
+                <sphere radius="0.05"/>
             </geometry>
         </collision>
@@ -115,3 +136,32 @@
         </xacro:inertial_sphere>
     </link>
+    <gazebo reference="caster_wheel_link">
+        <visual>
+            <material>
+                <ambient>0.1 0.1 0.1 1.0</ambient>
+                <diffuse>0.1 0.1 0.1 1.0</diffuse>
+                <specular>0.8 0.8 0.8 1.0</specular>
+            </material>
+        </visual>
+        <mu1 value="0.001"/>
+        <mu2 value="0.001"/>
+    </gazebo>
+<!--
+    <gazebo>
+        <plugin name="gz::sim::systems::DiffDrive" filename="gz-sim-diff-drive-system">
+            <left_joint>left_wheel_joint</left_joint>
+            <right_joint>right_wheel_joint</right_joint>
+            <wheel_separation>0.35</wheel_separation>
+            <wheel_radius>0.05</wheel_radius>
+            <topic>/cmd_vel</topic>
+            <frame_id>odom</frame_id>
+            <child_frame_id>base_link</child_frame_id>
+            <tf_topic>/tf</tf_topic>
+        </plugin>
+        <plugin name="gz::sim::systems::JointStatePublisher" filename="gz-sim-joint-state-publisher-system">
+            <joint>left_wheel_joint</joint>
+            <joint>right_wheel_joint</joint>
+        </plugin>
+    </gazebo>
+    -->
 </robot>
